Commit message: added my robot which is half the size of original bot

File: urdf/backup_lesson_bot/udacity_bot.xacro (robot description, xacro)
@@ -22,5 +22,5 @@
       <origin xyz="0 0 0" rpy=" 0 0 0"/>
       <geometry>
-        <box size=".2 .1 .05"/>
+        <box size=".4 .2 .1"/>
       </geometry>
     </collision>
@@ -28,5 +28,5 @@
       <origin xyz="0 0 0" rpy=" 0 0 0"/>
       <geometry>
-        <box size=".2 .1 .05"/>
+        <box size=".4 .2 .1"/>
       </geometry>
       <material name="Cyan">
@@ -35,7 +35,7 @@
     </visual>
     <collision name='back_caster_collision'>
-      <origin xyz="-0.075 0 -0.025" rpy=" 0 0 0"/>
-      <geometry>
-        <sphere radius="0.025"/>
+      <origin xyz="-0.15 0 -0.05" rpy=" 0 0 0"/>
+      <geometry>
+        <sphere radius="0.045"/>
       </geometry>
       <surface>
@@ -51,7 +51,7 @@
     </collision>
     <visual name='back_caster_visual'>
-      <origin xyz="-0.075 0 -0.025" rpy=" 0 0 0"/>
-      <geometry>
-        <sphere radius="0.025"/>
+      <origin xyz="-0.15 0 -0.05" rpy=" 0 0 0"/>
+      <geometry>
+        <sphere radius="0.045"/>
       </geometry>
       <material name="Cyan">
@@ -60,7 +60,7 @@
     </visual>
     <collision name='front_caster_collision'>
-      <origin xyz="0.075 0 -0.025" rpy=" 0 0 0"/>
-      <geometry>
-        <sphere radius="0.025"/>
+      <origin xyz="0.15 0 -0.05" rpy=" 0 0 0"/>
+      <geometry>
+        <sphere radius="0.045"/>
       </geometry>
       <surface>
@@ -76,7 +76,7 @@
     </collision>
     <visual name='front_caster_visual'>
-      <origin xyz="0.075 0 -0.025" rpy=" 0 0 0"/>
-      <geometry>
-        <sphere radius="0.025"/>
+      <origin xyz="0.15 0 -0.05" rpy=" 0 0 0"/>
+      <geometry>
+        <sphere radius="0.045"/>
       </geometry>
       <material name="Cyan">
@@ -98,11 +98,11 @@
       <origin xyz="0 0 0" rpy="0 1.5707 1.5707"/>
       <geometry>
-        <cylinder radius="0.05" length="0.025"/>
-      </geometry>
-    </collision>
-    <visual name='chassis_visual'>
-      <origin xyz="0 0 0" rpy="0 1.5707 1.5707"/>
-      <geometry>
-        <cylinder radius="0.05" length="0.025"/>
+        <cylinder radius="0.1" length="0.05"/>
+      </geometry>
+    </collision>
+    <visual name='chassis_visual'>
+      <origin xyz="0 0 0" rpy="0 1.5707 1.5707"/>
+      <geometry>
+        <cylinder radius="0.1" length="0.05"/>
       </geometry>
     </visual>
@@ -110,5 +110,5 @@
   <!--joint type="continuous" name="left_wheel_hinge"-->
   <joint type="continuous" name="left_wheel_hinge">
-    <origin xyz="0 0.075 0" rpy="0 0 0"/>
+    <origin xyz="0 0.15 0" rpy="0 0 0"/>
     <child link="left_wheel"/>
     <parent link="chassis"/>
@@ -130,11 +130,11 @@
       <origin xyz="0 0 0" rpy="0 1.5707 1.5707"/>
       <geometry>
-        <cylinder radius="0.05" length="0.025"/>
-      </geometry>
-    </collision>
-    <visual name='chassis_visual'>
-      <origin xyz="0 0 0" rpy="0 1.5707 1.5707"/>
-      <geometry>
-        <cylinder radius="0.05" length="0.025"/>
+        <cylinder radius="0.1" length="0.05"/>
+      </geometry>
+    </collision>
+    <visual name='chassis_visual'>
+      <origin xyz="0 0 0" rpy="0 1.5707 1.5707"/>
+      <geometry>
+        <cylinder radius="0.1" length="0.05"/>
       </geometry>
     </visual>
@@ -142,5 +142,5 @@
   <!--joint type="continuous" name="left_wheel_hinge"-->
   <joint type="continuous" name="right_wheel_hinge">
-    <origin xyz="0 -0.075 0" rpy="0 0 0"/>
+    <origin xyz="0 -0.15 0" rpy="0 0 0"/>
     <child link="right_wheel"/>
     <parent link="chassis"/>
@@ -163,11 +163,11 @@
       <origin xyz="0 0 0" rpy="0 0 0"/>
       <geometry>
-        <box size="0.025 0.025 0.025"/>
-      </geometry>
-    </collision>
-    <visual name='chassis_visual'>
-      <origin xyz="0 0 0" rpy="0 0 0"/>
-      <geometry>
-        <box size="0.025 0.025 0.025"/>
+        <box size="0.05 0.05 0.05"/>
+      </geometry>
+    </collision>
+    <visual name='chassis_visual'>
+      <origin xyz="0 0 0" rpy="0 0 0"/>
+      <geometry>
+        <box size="0.05 0.05 0.05"/>
       </geometry>
       <material name="Cyan">
@@ -178,5 +178,5 @@
   <!--joint type="continuous" name="left_wheel_hinge"-->
   <joint type="fixed" name="camera_joint">
-    <origin xyz="0.1 0 0" rpy="0 0 0"/>
+    <origin xyz="0.2 0 0" rpy="0 0 0"/>
     <child link="camera"/>
     <parent link="chassis"/>
@@ -207,5 +207,5 @@
   </link>
   <joint type="fixed" name="hokuyo_joint">
-    <origin xyz="0.075 0 0.05" rpy="0 0 0"/>
+    <origin xyz="0.15 0 0.1" rpy="0 0 0"/>
     <child link="hokuyo"/>
     <parent link="chassis"/>
